Commit message: Add package and update URDF model
The added package (romaa_gazebo) has a launch file to spawn
the robot model in the Gazebo simulator.

The URDF robot model of 'romaa_description' package was
modified to include the simulation parameters.

File: romaa_description/urdf/romaa.urdf (robot description, URDF)
Before this commit: robot romaa, 1 links, 0 joints
Links:
- link base_link: mass None -> 5; geometry collision box size=0.57 0.52 0.006; visual mesh filename=package://romaa_description/meshes/romaa_bottom.stl

Commit message: Update dynamic parameters of robot model

File: romaa_description/urdf/romaa.urdf (robot description, URDF)
Before this commit: robot romaa, 1 links, 0 joints
Links:
- link base_link: mass 5 -> 4.03317563367091

Commit message: Add robot columns to URDF model (only for RViz)

File: romaa_description/urdf/romaa.urdf (robot description, URDF)
Before this commit: robot romaa, 1 links, 0 joints
Links:
- added link fleft_column_link; visual cylinder length=0.154 radius=0.008
- added link fright_column_link; visual cylinder length=0.154 radius=0.008
- added link left_column_link; visual box size=0.050 0.015 0.154
- added link right_column_link; visual box size=0.050 0.015 0.154
- added link rleft_column_link; visual cylinder length=0.154 radius=0.008
- added link rright_column_link; visual cylinder length=0.154 radius=0.008
Joints:
- added joint fleft_column_joint: type fixed, parent base_link, child fleft_column_link, origin xyz=0.164 0.139 0.083 rpy=0 0 0
- added joint fright_column_joint: type fixed, parent base_link, child fright_column_link, origin xyz=0.164 -0.139 0.083 rpy=0 0 0
- added joint left_column_joint: type fixed, parent base_link, child left_column_link, origin xyz=-0.0835 0.250 0.083 rpy=0 0 0
- added joint right_column_joint: type fixed, parent base_link, child right_column_link, origin xyz=-0.0835 -0.250 0.083 rpy=0 0 0
- added joint rleft_column_joint: type fixed, parent base_link, child rleft_column_link, origin xyz=-0.337 0.212 0.083 rpy=0 0 0
- added joint rright_column_joint: type fixed, parent base_link, child rright_column_link, origin xyz=-0.337 -0.212 0.083 rpy=0 0 0
