Commit message: Update robot model to include Gazebo description

File: romaa_description/urdf/columns.xacro (robot description, xacro)
@@ -1,4 +1,20 @@
 <?xml version='1.0'?>
 <robot xmlns:xacro="http://www.ros.org/wiki/xacro">
+  <xacro:property name="D" value="2700" />   <!-- [Kg/m3] -->
+  <xacro:property name="h" value="0.154" /> <!-- [m] -->
+  <xacro:property name="r" value="0.008" /> <!-- [m] -->
+  <xacro:property name="w" value="0.050" /> <!-- [m] -->
+  <xacro:property name="d" value="0.015" /> <!-- [m] -->
+  <!-- Main column properties -->
+  <xacro:property name="mc_volume" value="${h * w * d}" />
+  <xacro:property name="mc_mass" value="${mc_volume * D}" />
+  <xacro:property name="mc_ixx" value="${(1/12) * mc_mass * (d**2 + h**2)}" />
+  <xacro:property name="mc_iyy" value="${(1/12) * mc_mass * (w**2 + h**2)}" />
+  <xacro:property name="mc_izz" value="${(1/12) * mc_mass * (d**2 + w**2)}" />
+  <!-- Secondary column properties -->
+  <xacro:property name="sc_volume" value="${pi * r**2 * h}" />
+  <xacro:property name="sc_mass" value="${sc_volume * D}" />
+  <xacro:property name="sc_ixx_yy" value="${(1/12) * sc_mass * h**2}" />
+  <xacro:property name="sc_izz" value="${(1/2) * sc_mass * r**2}" />
   <!-- Macro for robot main columns -->
   <xacro:macro name="main_column" params="name origin_xyz">
@@ -7,8 +23,20 @@
         <origin xyz="0 0 0" rpy="0 0 0" />
         <geometry>
-          <box size="0.050 0.015 0.154" />
+          <box size="${w} ${d} ${h}" />
         </geometry>
         <material name="black" />
       </visual>
+      <inertial>
+        <origin xyz="0 0 ${h / 2}" rpy="0 0 0" />
+        <mass value="${mc_mass}" />
+        <inertia ixx="${mc_ixx}" ixy="0" ixz="0"
+            iyy="${mc_iyy}" iyz="0" izz="${mc_izz}" />
+      </inertial>
+      <collision name="collision_base_link">
+        <origin xyz="0 0 0" rpy="0 0 0" />
+        <geometry>
+          <box size="${w} ${d} ${h}" />
+        </geometry>
+      </collision>
     </link>
     <joint name="${name}_joint" type="fixed">
@@ -24,8 +52,20 @@
         <origin xyz="0 0 0" rpy="0 0 0" />
         <geometry>
-          <cylinder length="0.154" radius="0.008" />
+          <cylinder length="${h}" radius="${r}" />
         </geometry>
         <material name="black" />
       </visual>
+      <inertial>
+        <origin xyz="0 0 ${h / 2}" rpy="0 0 0" />
+        <mass value="${sc_mass}" />
+        <inertia ixx="${sc_ixx_yy}" ixy="0" ixz="0"
+            iyy="${sc_ixx_yy}" iyz="0" izz="${sc_izz}" />
+      </inertial>
+      <collision name="collision_base_link">
+        <origin xyz="0 0 ${h / 2}" rpy="0 0 0" />
+        <geometry>
+          <cylinder length="${h}" radius="${r}" />
+        </geometry>
+      </collision>
     </link>
     <joint name="${name}_joint" type="fixed">

File: romaa_description/urdf/romaa.xacro (robot description, xacro)
@@ -2,4 +2,5 @@
 <robot name="romaa" xmlns:xacro="http://www.ros.org/wiki/xacro">
   <xacro:include filename="$(find romaa_description)/urdf/columns.xacro" />
+  <xacro:include filename="$(find romaa_description)/urdf/romaa.gazebo" />
   <material name="blue">
     <color rgba="0 0 0.8 1" />
@@ -8,7 +9,4 @@
     <color rgba="0.05 0.05 0.05 1" />
   </material>
-  <gazebo reference="base_link">
-    <material>Gazebo/Blue</material>
-  </gazebo>
   <!-- Base Link (bottom) -->
   <link name="base_link">
@@ -22,7 +20,7 @@
     <inertial>
       <origin xyz="0 0 0.003" rpy="0 0 0" />
-      <mass value="4.03317563367091"/>
-      <inertia ixx="0.0729296621571746" ixy="0" ixz="0"
-        iyy="0.0944958177861172" iyz="0" izz="0.16740128088949"/>
+      <mass value="4.115922297947584"/>
+      <inertia ixx="0.07709942829583775" ixy="0" ixz="0"
+        iyy="0.09727669030336457" iyz="0" izz="0.17435142306541462"/>
     </inertial>
     <collision name="collision_base_link">

Commit message: Fix offset in collision model and update doc

File: romaa_description/urdf/columns.xacro (robot description, xacro)
@@ -63,5 +63,5 @@
       </inertial>
       <collision name="collision_base_link">
-        <origin xyz="0 0 ${h / 2}" rpy="0 0 0" />
+        <origin xyz="0 0 0" rpy="0 0 0" />
         <geometry>
           <cylinder length="${h}" radius="${r}" />

Commit message: Add castor wheel support to robot model

File: romaa_description/urdf/columns.xacro (robot description, xacro)
@@ -6,4 +6,5 @@
   <xacro:property name="w" value="0.050" /> <!-- [m] -->
   <xacro:property name="d" value="0.015" /> <!-- [m] -->
+  <xacro:property name="c" value="0.03363" /> <!-- [m] -->
   <!-- Main column properties -->
   <xacro:property name="mc_volume" value="${h * w * d}" />
@@ -17,4 +18,9 @@
   <xacro:property name="sc_ixx_yy" value="${(1/12) * sc_mass * h**2}" />
   <xacro:property name="sc_izz" value="${(1/2) * sc_mass * r**2}" />
+  <!-- Castor column properties -->
+  <xacro:property name="cc_volume" value="${pi * r**2 * c}" />
+  <xacro:property name="cc_mass" value="${cc_volume * D}" />
+  <xacro:property name="cc_ixx_yy" value="${(1/12) * sc_mass * c**2}" />
+  <xacro:property name="cc_izz" value="${(1/2) * sc_mass * r**2}" />
   <!-- Macro for robot main columns -->
   <xacro:macro name="main_column" params="name origin_xyz">
@@ -33,5 +39,5 @@
             iyy="${mc_iyy}" iyz="0" izz="${mc_izz}" />
       </inertial>
-      <collision name="collision_base_link">
+      <collision>
         <origin xyz="0 0 0" rpy="0 0 0" />
         <geometry>
@@ -62,5 +68,5 @@
             iyy="${sc_ixx_yy}" iyz="0" izz="${sc_izz}" />
       </inertial>
-      <collision name="collision_base_link">
+      <collision>
         <origin xyz="0 0 0" rpy="0 0 0" />
         <geometry>
@@ -75,3 +81,32 @@
     </joint>
   </xacro:macro>
+  <!-- Macro for robot castor columns -->
+  <xacro:macro name="castor_column" params="name origin_xyz">
+    <link name="${name}_link">
+      <visual>
+        <origin xyz="0 0 0" rpy="0 0 0" />
+        <geometry>
+          <cylinder length="${c}" radius="${r}" />
+        </geometry>
+        <material name="black" />
+      </visual>
+      <inertial>
+        <origin xyz="0 0 ${c / 2}" rpy="0 0 0" />
+        <mass value="${cc_mass}" />
+        <inertia ixx="${cc_ixx_yy}" ixy="0" ixz="0"
+            iyy="${cc_ixx_yy}" iyz="0" izz="${cc_izz}" />
+      </inertial>
+      <collision>
+        <origin xyz="0 0 0" rpy="0 0 0" />
+        <geometry>
+          <cylinder length="${c}" radius="${r}" />
+        </geometry>
+      </collision>
+    </link>
+    <joint name="${name}_joint" type="fixed">
+      <parent link="base_link" />
+      <child link="${name}_link" />
+      <origin xyz="${origin_xyz}" rpy="0 0 0" />
+    </joint>
+  </xacro:macro>
 </robot>

File: romaa_description/urdf/romaa.xacro (robot description, xacro)
@@ -35,9 +35,13 @@
   <!-- Right main column -->
   <xacro:main_column name="right_column" origin_xyz="-0.0835 -0.250 0.083" />
-  <!-- Front-left column -->
+  <!-- Secondary columns -->
   <xacro:secondary_column name="fleft_column" origin_xyz="0.164 0.139 0.083" />  <!-- Front-left -->
   <xacro:secondary_column name="fright_column" origin_xyz="0.164 -0.139 0.083" />  <!-- Front-right -->
   <xacro:secondary_column name="rleft_column" origin_xyz="-0.337 0.212 0.083" />  <!-- Rear-left -->
   <xacro:secondary_column name="rright_column" origin_xyz="-0.337 -0.212 0.083" />  <!-- Rear-right -->
+  <!-- Castor support columns -->
+  <xacro:castor_column name="fc_column" origin_xyz="-0.332  0    0.022815" />
+  <xacro:castor_column name="lc_column" origin_xyz="-0.380 -0.06 0.022815" />
+  <xacro:castor_column name="rc_column" origin_xyz="-0.380  0.06 0.022815" />
   <!-- Top-front link -->
   <link name="top_front_link">
@@ -94,3 +98,30 @@
     <origin xyz="-0.236 0 0.160" rpy="0 0 0" />
   </joint>
+  <!-- Castor support link -->
+  <link name="csupport_link">
+    <visual>
+      <origin xyz="0 0 0" rpy="0 0 0" />
+      <geometry>
+        <mesh filename="package://romaa_description/meshes/romaa_castor_support.stl" />
+      </geometry>
+      <material name="blue" />
+    </visual>
+    <inertial>
+      <origin xyz="0 0 0.003" rpy="0 0 0" />
+      <mass value="0.190755"/>
+      <inertia ixx="0.00023339157749999997" ixy="0" ixz="0"
+        iyy="0.00014052256237261147" iyz="0" izz="0.0003727696098726115"/>
+    </inertial>
+    <collision name="collision_base_link">
+      <origin xyz="0 0 0.003" rpy="0 0 0" />
+      <geometry>
+        <box size="0.105 0.140 0.006"/>
+      </geometry>
+    </collision>
+  </link>
+  <joint name="csupport_joint" type="fixed">
+    <parent link="base_link" />
+    <child link="csupport_link" />
+    <origin xyz="-0.378 0 0.03963" rpy="0 0 0" />
+  </joint>
 </robot>
