Commit message: Correct robot floor clearance

File: romaa_description/urdf/wheels.xacro (robot description, xacro)
@@ -5,5 +5,5 @@
   <xacro:property name="wheel_radius" value="0.070" />
   <xacro:property name="wheel_thickness" value="0.025" />
-  <xacro:property name="wheel_zsep" value="0.037" />
+  <xacro:property name="wheel_zsep" value="0.033" />
   <!-- Macro for robot wheels -->
   <xacro:macro name="wheel" params="name reflect">
@@ -35,5 +35,4 @@
       <child link="${name}_link" />
       <axis xyz="0 1 0" />
-      <joint_properties damping="1.0" friction="1.0" />
     </joint>
   </xacro:macro>
