Commit message: Correct center of mass of robot parts

File: romaa_description/urdf/castor_wheel.xacro (robot description, xacro)
@@ -35,23 +35,23 @@
         <origin xyz="0 0 0" rpy="0 0 0" />
         <geometry>
-          <mesh filename="package://romaa_description/meshes/romaa_castor_base.stl" />
+          <mesh filename="package://romaa_description/meshes/romaa_castor_cylinder.stl" />
         </geometry>
         <material name="dark_gray" />
       </visual>
       <inertial>
-        <origin xyz="0 0 0" rpy="0 0 0" />
-        <mass value="0.022726972589783227" />
-        <inertia ixx="5.243689744256557e-06" ixy="0" ixz="0"
-            iyy="4.149252628753352e-06" iyz="0" izz="2.389246986591684e-06" />
+        <origin xyz="0.0048464279113944195 0 -0.0265" rpy="0 0 0" />
+        <mass value="0.03629327674887137" />
+        <inertia ixx="1.2058314484155499e-05" ixy="0" ixz="0"
+            iyy="9.601587537327375e-06" iyz="0" izz="6.537703376119888e-06" />
       </inertial>
       <collision>
         <origin xyz="0 0 -0.025" rpy="0 0 0" />
         <geometry>
-          <cylinder length="0.050" radius="0.012" />
+          <cylinder length="0.050" radius="0.030" />
         </geometry>
       </collision>
     </link>
     <joint name="${name}_rot1_joint" type="continuous">
-      <dynamics damping="0" friction="0.5" />
+      <!-- <dynamics damping="0" friction="0.2" /> -->
       <origin xyz="0 0 0.00075" rpy="0 0 0" />
       <parent link="${name}_b1_link" />
@@ -82,5 +82,5 @@
     </link>
     <joint name="${name}_rot2_joint" type="continuous">
-      <dynamics damping="0" friction="1" />
+      <dynamics damping="0" friction="0.2" />
       <origin xyz="-0.026 0 -0.04363" rpy="0 0 0" />
       <parent link="${name}_b2_link" />

File: romaa_description/urdf/drive_wheels.xacro (robot description, xacro)
@@ -18,8 +18,8 @@
       </visual>
       <inertial>
-        <origin xyz="0 0 0" rpy="0 0 0" />
+        <origin xyz="0 0 0" rpy="${pi / 2} 0 0" />
         <mass value="0.200" />
         <inertia ixx="0.0003179237060191715" ixy="0" ixz="0"
-            iyy="0.0006167682575358206" iyz="0" izz="0.00031792370601916626" />
+            iyy="0.00031792370601916626" iyz="0" izz="0.0006167682575358206" />
       </inertial>
       <collision>
@@ -31,6 +31,5 @@
     </link>
     <joint name="${name}_joint" type="continuous">
-      <dynamics damping="1.0" friction="1.0" />
-      <!-- <origin xyz="0 ${reflect * wheelbase / 2}" rpy="${pi} 0 0" /> -->
+      <!-- <dynamics damping="0.1" friction="0.1" />  -->
       <origin xyz="0 ${reflect * wheelbase / 2} ${wheel_zsep}" rpy="0 0 0" />
       <parent link="base_link" />

File: romaa_description/urdf/romaa.xacro (robot description, xacro)
@@ -2,7 +2,7 @@
 <robot name="romaa" xmlns:xacro="http://www.ros.org/wiki/xacro">
   <xacro:include filename="$(find romaa_description)/urdf/columns.xacro" />
-  <xacro:include filename="$(find romaa_description)/urdf/romaa.gazebo" />
   <xacro:include filename="$(find romaa_description)/urdf/drive_wheels.xacro" />
   <xacro:include filename="$(find romaa_description)/urdf/castor_wheel.xacro" />
+  <xacro:include filename="$(find romaa_description)/urdf/romaa.gazebo" />
   <material name="blue">
     <color rgba="0 0 0.8 1" />
@@ -27,5 +27,5 @@
     </visual>
     <inertial>
-      <origin xyz="0 0 0.003" rpy="0 0 0" />
+      <origin xyz="-0.10442512118169343 0 0.003" rpy="0 0 0" />
       <mass value="4.115922297947584"/>
       <inertia ixx="0.07709942829583775" ixy="0" ixz="0"
@@ -35,5 +35,5 @@
       <origin xyz="-0.111 0 0.003" rpy="0 0 0" />
       <geometry>
-        <box size="0.57 0.52 0.006"/>
+        <box size="0.570 0.520 0.006"/>
       </geometry>
     </collision>
@@ -44,8 +44,8 @@
   <xacro:main_column name="right_column" origin_xyz="-0.0835 -0.250 0.083" />
   <!-- Secondary columns -->
-  <xacro:secondary_column name="fleft_column" origin_xyz="0.164 0.139 0.083" />  <!-- Front-left -->
-  <xacro:secondary_column name="fright_column" origin_xyz="0.164 -0.139 0.083" />  <!-- Front-right -->
-  <xacro:secondary_column name="rleft_column" origin_xyz="-0.337 0.212 0.083" />  <!-- Rear-left -->
-  <xacro:secondary_column name="rright_column" origin_xyz="-0.337 -0.212 0.083" />  <!-- Rear-right -->
+  <xacro:secondary_column name="fleft_column" origin_xyz="0.164 0.139 0.083" />
+  <xacro:secondary_column name="fright_column" origin_xyz="0.164 -0.139 0.083" />
+  <xacro:secondary_column name="rleft_column" origin_xyz="-0.337 0.212 0.083" />
+  <xacro:secondary_column name="rright_column" origin_xyz="-0.337 -0.212 0.083" />
   <!-- Castor support columns -->
   <xacro:castor_column name="fc_column" origin_xyz="-0.332  0    0.022815" />
@@ -116,5 +116,5 @@
     </visual>
     <inertial>
-      <origin xyz="0 0 0.003" rpy="0 0 0" />
+      <origin xyz="0.0035 0 0.003" rpy="0 0 0" />
       <mass value="0.190755"/>
       <inertia ixx="0.00023339157749999997" ixy="0" ixz="0"
@@ -134,5 +134,4 @@
   </joint>
   <!-- Battery link -->
-  <!--
   <link name="battery_link">
     <visual>
@@ -161,5 +160,4 @@
     <origin xyz="-0.209 0 0.0685" rpy="0 0 0" />
   </joint>
-  -->
   <!-- Left drive wheel -->
   <xacro:drive_wheel name="left_wheel" reflect="1" />
@@ -167,6 +165,4 @@
   <xacro:drive_wheel name="right_wheel" reflect="-1" />
   <!-- Castor wheel -->
-  <!--
   <xacro:castor_wheel name="castor" origin_xyz="-0.016 0 -0.00075" />
-  -->
 </robot>

Commit message: Add friction to wheel surfaces

File: romaa_description/urdf/castor_wheel.xacro (robot description, xacro)
@@ -53,5 +53,5 @@
     </link>
     <joint name="${name}_rot1_joint" type="continuous">
-      <!-- <dynamics damping="0" friction="0.2" /> -->
+      <dynamics damping="0" friction="1.0" />
       <origin xyz="0 0 0.00075" rpy="0 0 0" />
       <parent link="${name}_b1_link" />
@@ -82,5 +82,5 @@
     </link>
     <joint name="${name}_rot2_joint" type="continuous">
-      <dynamics damping="0" friction="0.2" />
+      <!-- <dynamics damping="0" friction="0.5" /> -->
       <origin xyz="-0.026 0 -0.04363" rpy="0 0 0" />
       <parent link="${name}_b2_link" />

File: romaa_description/urdf/romaa.xacro (robot description, xacro)
@@ -134,4 +134,5 @@
   </joint>
   <!-- Battery link -->
+  <!--
   <link name="battery_link">
     <visual>
@@ -160,4 +161,5 @@
     <origin xyz="-0.209 0 0.0685" rpy="0 0 0" />
   </joint>
+  -->
   <!-- Left drive wheel -->
   <xacro:drive_wheel name="left_wheel" reflect="1" />

Commit message: Adjust wheel surface contact parameters

File: romaa_description/urdf/castor_wheel.xacro (robot description, xacro)
@@ -1,6 +1,12 @@
 <?xml version='1.0'?>
 <robot xmlns:xacro="http://www.ros.org/wiki/xacro">
+  <xacro:property name="b1_L" value="0.05" />
+  <xacro:property name="b1_H" value="0.0015" />
+  <xacro:property name="csupport_H" value="0.06863" />
+  <xacro:property name="b2_H" value="0.050" />
+  <xacro:property name="R_rueda" value="0.0245" />
+  <xacro:property name="z" value="${csupport_H - (b2_H/2) - b1_H - R_rueda}" />
   <!-- Macro for castor wheel -->
-  <xacro:macro name="castor_wheel" params="name origin_xyz">
+  <xacro:macro name="castor_wheel" params="name origin_x">
     <!-- Castor wheel base (cube) -->
     <link name="${name}_b1_link">
@@ -8,5 +14,5 @@
         <origin xyz="0 0 0" rpy="0 0 0" />
         <geometry>
-          <box size="0.05 0.05 0.0015" />
+          <box size="${b1_L} ${b1_L} ${b1_H}" />
         </geometry>
         <material name="dark_gray" />
@@ -26,5 +32,5 @@
     </link>
     <joint name="${name}_b1_joint" type="fixed">
-      <origin xyz="${origin_xyz}" rpy="0 0 0" />
+      <origin xyz="${origin_x} 0 -${b1_H / 2}" rpy="0 0 0" />
       <parent link="csupport_link" />
       <child link="${name}_b1_link" />
@@ -40,5 +46,5 @@
       </visual>
       <inertial>
-        <origin xyz="0.0048464279113944195 0 -0.0265" rpy="0 0 0" />
+        <origin xyz="0.0048464279113944195 0 0" rpy="0 0 0" />
         <mass value="0.03629327674887137" />
         <inertia ixx="1.2058314484155499e-05" ixy="0" ixz="0"
@@ -46,13 +52,13 @@
       </inertial>
       <collision>
-        <origin xyz="0 0 -0.025" rpy="0 0 0" />
+        <origin xyz="0 0 0" rpy="0 0 0" />
         <geometry>
-          <cylinder length="0.050" radius="0.030" />
+          <cylinder length="${b2_H}" radius="0.030" />
         </geometry>
       </collision>
     </link>
     <joint name="${name}_rot1_joint" type="continuous">
-      <dynamics damping="0" friction="1.0" />
-      <origin xyz="0 0 0.00075" rpy="0 0 0" />
+      <dynamics damping="0.0" friction="0.5" />
+      <origin xyz="0 0 -${(b1_H/2) + (b2_H/2)}" rpy="0 0 0" />
       <parent link="${name}_b1_link" />
       <child link="${name}_b2_link" />
@@ -69,5 +75,5 @@
       </visual>
       <inertial>
-        <origin xyz="0 0 0" rpy="0 0 0" />
+        <origin xyz="0 0 0" rpy="${pi / 2} 0 0" />
         <mass value="0.0233673699785761" />
         <inertia ixx="4.260422817439314e-06" ixy="0" ixz="0"
@@ -82,6 +88,6 @@
     </link>
     <joint name="${name}_rot2_joint" type="continuous">
-      <!-- <dynamics damping="0" friction="0.5" /> -->
-      <origin xyz="-0.026 0 -0.04363" rpy="0 0 0" />
+      <dynamics damping="0.0" friction="0.5" />
+      <origin xyz="-0.026 0 -${z}" rpy="0 0 0" />
       <parent link="${name}_b2_link" />
       <child link="${name}_link" />

File: romaa_description/urdf/drive_wheels.xacro (robot description, xacro)
@@ -31,5 +31,5 @@
     </link>
     <joint name="${name}_joint" type="continuous">
-      <!-- <dynamics damping="0.1" friction="0.1" />  -->
+      <dynamics damping="0.1" friction="0.5" />
       <origin xyz="0 ${reflect * wheelbase / 2} ${wheel_zsep}" rpy="0 0 0" />
       <parent link="base_link" />

File: romaa_description/urdf/romaa.xacro (robot description, xacro)
@@ -134,8 +134,7 @@
   </joint>
   <!-- Battery link -->
-  <!--
   <link name="battery_link">
     <visual>
-      <origin xyz="0 0 0" rpy="0 0 ${-pi / 2}" />
+      <origin xyz="0 0 0" rpy="0 0 0" />
       <geometry>
         <box size="0.175 0.166 0.125"/>
@@ -144,5 +143,5 @@
     </visual>
     <inertial>
-      <origin xyz="0 0 0" rpy="0 0 ${-pi / 2}" />
+      <origin xyz="0 0 0" rpy="0 0 0" />
       <mass value="11.467"/>
       <inertia ixx="0.04126479814479167" ixy="0" ixz="0"
@@ -150,5 +149,5 @@
     </inertial>
     <collision>
-      <origin xyz="0 0 0" rpy="0 0 ${-pi / 2}" />
+      <origin xyz="0 0 0" rpy="0 0 0" />
       <geometry>
         <box size="0.175 0.166 0.125"/>
@@ -161,5 +160,4 @@
     <origin xyz="-0.209 0 0.0685" rpy="0 0 0" />
   </joint>
-  -->
   <!-- Left drive wheel -->
   <xacro:drive_wheel name="left_wheel" reflect="1" />
@@ -167,4 +165,4 @@
   <xacro:drive_wheel name="right_wheel" reflect="-1" />
   <!-- Castor wheel -->
-  <xacro:castor_wheel name="castor" origin_xyz="-0.016 0 -0.00075" />
+  <xacro:castor_wheel name="castor" origin_x="-0.016" />
 </robot>
