Commit message: Add top plates to the robot model

File: romaa_description/urdf/romaa.xacro (robot description, xacro)
@@ -9,5 +9,5 @@
     <color rgba="0.05 0.05 0.05 1" />
   </material>
-  <!-- Base Link (bottom) -->
+  <!-- Base link (bottom) -->
   <link name="base_link">
     <visual>
@@ -40,3 +40,57 @@
   <xacro:secondary_column name="rleft_column" origin_xyz="-0.337 0.212 0.083" />  <!-- Rear-left -->
   <xacro:secondary_column name="rright_column" origin_xyz="-0.337 -0.212 0.083" />  <!-- Rear-right -->
+  <!-- Top-front link -->
+  <link name="top_front_link">
+    <visual>
+      <origin xyz="0 0 0" rpy="0 0 0" />
+      <geometry>
+        <mesh filename="package://romaa_description/meshes/romaa_top_front.stl" />
+      </geometry>
+      <material name="blue" />
+    </visual>
+    <inertial>
+      <origin xyz="0 0 0.003" rpy="0 0 0" />
+      <mass value="0.7186369596364028"/>
+      <inertia ixx="0.014812833616776537" ixy="0" ixz="0"
+        iyy="0.003404563417864952" iyz="0" izz="0.018213085212883666"/>
+    </inertial>
+    <collision name="collision_base_link">
+      <origin xyz="0.049 0 0.003" rpy="0 0 0" />
+      <geometry>
+        <box size="0.250 0.520 0.006"/>
+      </geometry>
+    </collision>
+  </link>
+  <joint name="top_front_joint" type="fixed">
+    <parent link="base_link" />
+    <child link="top_front_link" />
+    <origin xyz="0 0 0.160" rpy="0 0 0" />
+  </joint>
+  <!-- Top-rear link -->
+  <link name="top_rear_link">
+    <visual>
+      <origin xyz="0 0 0" rpy="0 0 0" />
+      <geometry>
+        <mesh filename="package://romaa_description/meshes/romaa_top_rear.stl" />
+      </geometry>
+      <material name="blue" />
+    </visual>
+    <inertial>
+      <origin xyz="0 0 0.003" rpy="0 0 0" />
+      <mass value="0.8885077118205166"/>
+      <inertia ixx="0.016809690318237213" ixy="0" ixz="0"
+        iyy="0.007046759808520824" iyz="0" izz="0.02385111908048711"/>
+    </inertial>
+    <collision name="collision_base_link">
+      <origin xyz="0 0 0.003" rpy="0 0 0" />
+      <geometry>
+        <box size="0.320 0.520 0.006"/>
+      </geometry>
+    </collision>
+  </link>
+  <joint name="top_rear_joint" type="fixed">
+    <parent link="base_link" />
+    <child link="top_rear_link" />
+    <origin xyz="-0.236 0 0.160" rpy="0 0 0" />
+  </joint>
 </robot>

Commit message: Add battery to robot model

File: romaa_description/urdf/romaa.xacro (robot description, xacro)
@@ -8,4 +8,7 @@
   <material name="black">
     <color rgba="0.05 0.05 0.05 1" />
+  </material>
+  <material name="dark_gray">
+    <color rgba="0.12 0.12 0.12 1" />
   </material>
   <!-- Base link (bottom) -->
@@ -24,5 +27,5 @@
         iyy="0.09727669030336457" iyz="0" izz="0.17435142306541462"/>
     </inertial>
-    <collision name="collision_base_link">
+    <collision>
       <origin xyz="-0.111 0 0.003" rpy="0 0 0" />
       <geometry>
@@ -59,5 +62,5 @@
         iyy="0.003404563417864952" iyz="0" izz="0.018213085212883666"/>
     </inertial>
-    <collision name="collision_base_link">
+    <collision>
       <origin xyz="0.049 0 0.003" rpy="0 0 0" />
       <geometry>
@@ -86,5 +89,5 @@
         iyy="0.007046759808520824" iyz="0" izz="0.02385111908048711"/>
     </inertial>
-    <collision name="collision_base_link">
+    <collision>
       <origin xyz="0 0 0.003" rpy="0 0 0" />
       <geometry>
@@ -113,5 +116,5 @@
         iyy="0.00014052256237261147" iyz="0" izz="0.0003727696098726115"/>
     </inertial>
-    <collision name="collision_base_link">
+    <collision>
       <origin xyz="0 0 0.003" rpy="0 0 0" />
       <geometry>
@@ -125,3 +128,30 @@
     <origin xyz="-0.378 0 0.03963" rpy="0 0 0" />
   </joint>
+  <!-- Battery link -->
+  <link name="battery_link">
+    <visual>
+      <origin xyz="0 0 0" rpy="0 0 0" />
+      <geometry>
+        <box size="0.175 0.166 0.126"/>
+      </geometry>
+      <material name="dark_gray" />
+    </visual>
+    <inertial>
+      <origin xyz="0 0 0" rpy="0 0 0" />
+      <mass value="8.9"/>
+      <inertia ixx="0.032218760985599997" ixy="0" ixz="0"
+        iyy="0.0344954090208" iyz="0" izz="0.0431598759648"/>
+    </inertial>
+    <collision>
+      <origin xyz="0 0 0" rpy="0 0 0" />
+      <geometry>
+        <box size="0.175 0.166 0.126"/>
+      </geometry>
+    </collision>
+  </link>
+  <joint name="battery_joint" type="fixed">
+    <parent link="base_link" />
+    <child link="battery_link" />
+    <origin xyz="-0.19 0 0.069" rpy="0 0 0" />
+  </joint>
 </robot>

Commit message: Add drive wheels and gazebo diff-drive plugin

File: romaa_description/urdf/romaa.xacro (robot description, xacro)
@@ -3,4 +3,5 @@
   <xacro:include filename="$(find romaa_description)/urdf/columns.xacro" />
   <xacro:include filename="$(find romaa_description)/urdf/romaa.gazebo" />
+  <xacro:include filename="$(find romaa_description)/urdf/wheels.xacro" />
   <material name="blue">
     <color rgba="0 0 0.8 1" />
@@ -11,4 +12,7 @@
   <material name="dark_gray">
     <color rgba="0.12 0.12 0.12 1" />
+  </material>
+  <material name="light_gray">
+    <color rgba="0.4 0.4 0.4 1" />
   </material>
   <!-- Base link (bottom) -->
@@ -155,3 +159,7 @@
     <origin xyz="-0.19 0 0.069" rpy="0 0 0" />
   </joint>
+  <!-- Left wheel -->
+  <xacro:wheel name="left_wheel" reflect="1" />
+  <!-- Right wheel -->
+  <xacro:wheel name="right_wheel" reflect="-1" />
 </robot>

Commit message: Add laser rangefinder sensor

File: romaa_description/urdf/romaa.xacro (robot description, xacro)
@@ -5,4 +5,12 @@
   <xacro:include filename="$(find romaa_description)/urdf/castor_wheel.xacro" />
   <xacro:include filename="$(find romaa_description)/urdf/romaa.gazebo" />
+  <xacro:include filename="$(find romaa_description)/urdf/laser.gazebo" />
+  <xacro:arg name="laser_enabled" default="$(optenv ROMAA_LASER 0)" />
+  <xacro:property name="laser_min_dist" value="0.10" />
+  <xacro:property name="laser_max_dist" value="10.0" />
+  <xacro:property name="laser_samples" value="540" />
+  <xacro:property name="laser_resol" value="0.5" />
+  <xacro:property name="laser_min_angle" value="${-(3/4)*pi}" />
+  <xacro:property name="laser_max_angle" value="${(3/4)*pi}" />
   <material name="blue">
     <color rgba="0 0 0.8 1" />
@@ -16,4 +24,7 @@
   <material name="light_gray">
     <color rgba="0.4 0.4 0.4 1" />
+  </material>
+  <material name="gray">
+    <color rgba="0.8 0.8 .8 1" />
   </material>
   <!-- Base link (bottom) -->
@@ -134,4 +145,5 @@
   </joint>
   <!-- Battery link -->
+  <!--
   <link name="battery_link">
     <visual>
@@ -160,4 +172,5 @@
     <origin xyz="-0.209 0 0.0685" rpy="0 0 0" />
   </joint>
+  -->
   <!-- Left drive wheel -->
   <xacro:drive_wheel name="left_wheel" reflect="1" />
@@ -166,3 +179,33 @@
   <!-- Castor wheel -->
   <xacro:castor_wheel name="castor" origin_x="-0.016" />
+  <!-- Laser rangefinder sensor -->
+  <xacro:if value="$(arg laser_enabled)">
+    <link name="laser_link">
+      <visual>
+        <origin xyz="0 0 0" rpy="0 0 0" />
+        <geometry>
+          <mesh filename="package://romaa_description/meshes/hokuyo.dae" />
+        </geometry>
+        <material name="gray" />
+      </visual>
+      <collision>
+        <origin xyz="0 0 0" rpy="0 0 0"/>
+        <geometry>
+          <box size="0.05 0.05 0.07" />
+        </geometry>
+      </collision>
+      <inertial>
+        <mass value="1e-5" />
+        <origin xyz="0 0 0" rpy="0 0 0"/>
+        <inertia ixx="1e-6" ixy="0" ixz="0" iyy="1e-6" iyz="0" izz="1e-6" />
+      </inertial>
+    </link>
+    <joint name="joint_laser" type="fixed" >
+      <parent link="top_front_link" />
+      <child link="laser_link" />
+      <origin xyz="0.0 0 0.035" rpy="0 0 0" />
+    </joint>
+    <xacro:laser min_dist="${laser_min_dist}" max_dist="${laser_max_dist}" samples="${laser_samples}"
+        resol="${laser_resol}" min_angle="${laser_min_angle}" max_angle="${laser_max_angle}" />
+  </xacro:if>
 </robot>

Commit message: Add Gazebo world file

File: romaa_description/urdf/romaa.xacro (robot description, xacro)
@@ -10,5 +10,5 @@
   <xacro:property name="laser_max_dist" value="10.0" />
   <xacro:property name="laser_samples" value="540" />
-  <xacro:property name="laser_resol" value="0.5" />
+  <xacro:property name="laser_resol" value="1" />
   <xacro:property name="laser_min_angle" value="${-(3/4)*pi}" />
   <xacro:property name="laser_max_angle" value="${(3/4)*pi}" />

Commit message: Add sensor bar

File: romaa_description/urdf/romaa.xacro (robot description, xacro)
@@ -173,4 +173,31 @@
   </joint>
   -->
+  <!-- Sensor bar link -->
+  <link name="sensbar_link">
+    <visual>
+      <origin xyz="0 0 0" rpy="0 0 0" />
+      <geometry>
+        <mesh filename="package://romaa_description/meshes/romaa_sensor_bar_with_holes.stl" />
+      </geometry>
+      <material name="black" />
+    </visual>
+    <inertial>
+      <origin xyz="-0.17062558720045456 0 7.489880295179326" />
+      <mass value="0.6705571211803331"/>
+      <inertia ixx="0.006744639700932016" ixy="0" ixz="0"
+        iyy="0.00015281269307933294" iyz="0" izz="0.006872329258775596"/>
+    </inertial>
+    <collision>
+      <origin xyz="0 0 0" rpy="0 0 0" />
+      <geometry>
+        <mesh filename="package://romaa_description/meshes/romaa_sensor_bar.stl" />
+      </geometry>
+    </collision>
+  </link>
+  <joint name="sensor_bar_joint" type="fixed">
+    <parent link="top_front_link" />
+    <child link="sensbar_link" />
+    <origin xyz="0.129 0 0.006" rpy="0 0 0" />
+  </joint>
   <!-- Left drive wheel -->
   <xacro:drive_wheel name="left_wheel" reflect="1" />

Commit message: Add new model of laser rangefinder sensor

File: romaa_description/urdf/romaa.xacro (robot description, xacro)
@@ -7,4 +7,6 @@
   <xacro:include filename="$(find romaa_description)/urdf/laser.gazebo" />
   <xacro:arg name="laser_enabled" default="false" />
+  <xacro:arg name="laser_on_bar" default="false" />
+  <!-- Laser rangefinder properties -->
   <xacro:property name="laser_min_dist" value="0.10" />
   <xacro:property name="laser_max_dist" value="10.0" />
@@ -212,5 +214,5 @@
         <origin xyz="0 0 0" rpy="0 0 0" />
         <geometry>
-          <mesh filename="package://romaa_description/meshes/hokuyo.dae" />
+          <mesh filename="package://romaa_description/meshes/sick_tim_1xxx.stl" />
         </geometry>
         <material name="gray" />
@@ -231,5 +233,16 @@
       <parent link="top_front_link" />
       <child link="laser_link" />
-      <origin xyz="0.0 0 0.035" rpy="0 0 0" />
+      <xacro:if value="$(arg laser_on_bar)">
+        <!-- Hokuyo laser rangefinder -->
+        <!--<origin xyz="0.129 0 0.056" rpy="0 0 0" />-->
+        <!-- Sick laser rangefinder -->
+        <origin xyz="0.129 0 0.084" rpy="0 0 0" />
+      </xacro:if>
+      <xacro:unless value="$(arg laser_on_bar)">
+        <!-- Hokuyo laser rangefinder -->
+        <!--<origin xyz="0.0 0 0.041" rpy="0 0 0" />-->
+        <!-- Sick laser rangefinder -->
+        <origin xyz="0.0 0 0.069" rpy="0 0 0" />
+      </xacro:unless>
     </joint>
     <xacro:laser min_dist="${laser_min_dist}" max_dist="${laser_max_dist}" samples="${laser_samples}"
